File: hardware/PCB/hakea-fillets.kicad_sch (KiCad schematic)
At the start: 103 parts, among them J1 Conn_01x04_Female, J2 USB_C_Receptacle_USB2.0, J3 Conn_01x04_MountingPin, J4 Conn_01x03, Q1 AO3401A, SW1 SW_SPST, SW10 SW_Push, SW11 SW_Push, SW12 SW_Push, SW13 SW_Push, SW14 SW_Push, SW15 SW_Push, SW16 SW_Push, SW17 SW_Push, SW18 SW_Push, SW19 SW_Push, SW2 SW_Push, SW20 SW_Push, SW21 SW_Push, SW22 SW_Push, SW23 SW_Push, SW24 SW_Push, SW25 SW_Push, SW26 SW_Push, SW27 SW_Push, SW28 SW_Push, SW29 SW_Push, SW3 SW_Push, SW30 SW_Push, SW31 Rotary_Encoder_Switch, SW32 Rotary_Encoder_Switch, SW33 SW_SPDT, SW34 Rotary_Encoder_Switch, SW4 SW_Push, SW5 SW_Push, SW6 SW_Push, SW7 SW_Push, SW8 SW_Push, SW9 SW_Push, U1 AP2112K-3.3, U2 TP4054, U4 nRF52840_holyiot_18010

Commit message: Updates with license
Parts:
- gave numbers to parts that had none: 4
Connections:
- net at D1.1 (K), Q1.2 (S), U1.1 (VIN)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: no longer C3.1
Other:
- company: (none) -> TKW
- title: (none) -> Hakea Wireless Keyboard
- moved on the sheet: C3, C4, D1, D4, Q1, R2, R6, R7, R8, R9, SW1

Commit message: choco
Parts:
- J1: value Conn_01x04_Female -> SWD PORT
Connections:
- net GND: now also J3.MP (MountPin)
- net at D1.1 (K), Q1.2 (S), U1.1 (VIN)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: now also C3.1
- no-connect marks 0 -> 28
Other:
- moved on the sheet: C4, D2, R1, R5, R6
