File: hardware/PCB/hakea-fillets.kicad_sch (KiCad schematic)
At the start: 103 parts, among them J1 Conn_01x04_Female, J2 USB_C_Receptacle_USB2.0, J3 Conn_01x04_MountingPin, J4 Conn_01x03, Q1 AO3401A, SW1 SW_SPST, SW10 SW_Push, SW11 SW_Push, SW12 SW_Push, SW13 SW_Push, SW14 SW_Push, SW15 SW_Push, SW16 SW_Push, SW17 SW_Push, SW18 SW_Push, SW19 SW_Push, SW2 SW_Push, SW20 SW_Push, SW21 SW_Push, SW22 SW_Push, SW23 SW_Push, SW24 SW_Push, SW25 SW_Push, SW26 SW_Push, SW27 SW_Push, SW28 SW_Push, SW29 SW_Push, SW3 SW_Push, SW30 SW_Push, SW31 Rotary_Encoder_Switch, SW32 Rotary_Encoder_Switch, SW33 SW_SPDT, SW34 Rotary_Encoder_Switch, SW4 SW_Push, SW5 SW_Push, SW6 SW_Push, SW7 SW_Push, SW8 SW_Push, SW9 SW_Push, U1 AP2112K-3.3, U2 TP4054, U4 nRF52840_holyiot_18010

Commit message: Updates
Parts:
- C1: JLC Part (none) -> C1779; LCSC Part (none) -> C1779
- C2, C3: JLC Part (none) -> C28323; LCSC Part (none) -> C28323
- C4: JLC Part (none) -> C377103; LCSC Part (none) -> C377103
- D1: JLC Part (none) -> C963381; LCSC Part (none) -> C963381
- D10, D11, D12, D13, D14, D15, D16, D17, D18, D19, D20, D21, D22, D23, D24, D25, D26, D27, D28, D29, D30, D31, D32, D33, D34, D5, D6, D7, D8, D9: JLC Part (none) -> C81598; LCSC Part (none) -> C81598
- D2: JLC Part (none) -> C521962; LCSC Part (none) -> C521962
- D3, D4: JLC Part (none) -> C84256; LCSC Part (none) -> C84256
- F1: JLC Part (none) -> C75464; LCSC Part (none) -> C75464
- Q1: JLC Part (none) -> C15127; LCSC Part (none) -> C15127
- R1, R5: JLC Part (none) -> C104384; LCSC Part (none) -> C104384
- R2, R3: JLC Part (none) -> C165963; LCSC Part (none) -> C165963
- R6: JLC Part (none) -> C212286; LCSC Part (none) -> C212286
