File: hardware/PCB/hakea-choc.kicad_sch (KiCad schematic)
At the start: 99 parts, among them J1 SWD PORT, J2 USB_C_Receptacle_USB2.0, J3 epaper-102, J4 Conn_01x03, Q1 AO3401A, Q2 2N7002, Q3 AO3401A, SW1 SW_SPST, SW10 SW_Push, SW11 SW_Push, SW12 SW_Push, SW13 SW_Push, SW14 SW_Push, SW15 SW_Push, SW16 SW_Push, SW17 SW_Push, SW18 SW_Push, SW19 SW_Push, SW2 SW_Push, SW20 SW_Push, SW21 SW_Push, SW22 SW_Push, SW23 SW_Push, SW24 SW_Push, SW25 SW_Push, SW26 SW_Push, SW27 SW_Push, SW28 SW_Push, SW29 SW_Push, SW3 SW_Push, SW30 SW_Push, SW32 Rotary_Encoder_Switch, SW33 SW_SPDT, SW34 Rotary_Encoder_Switch, SW4 SW_Push, SW5 SW_Push, SW6 SW_Push, SW7 SW_Push, SW8 SW_Push, SW9 SW_Push, U1 AP2112K-3.3, U2 TP4054, U4 nRF52840_holyiot_18010

Commit message: WIP
Connections:
- net GND: now also Q2.2 (S), R11.1
Changed lines of the file:
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@@
   (junction (at 123.952 160.782) (diameter 1.016) (color 0 0 0 0)
   )
+  (junction (at 266.954 187.706) (diameter 0) (color 0 0 0 0)
+  )
   (junction (at 140.462 145.542) (diameter 1.016) (color 0 0 0 0)
   )
@@
     (pin "2")
   )
+  (symbol (lib_id "power:GND") (at 266.954 187.706 0) (unit 1)
+    (in_bom yes) (on_board yes)
+    (property "Reference" "#PWR?" (id 0) (at 266.954 194.056 0)
+      (effects (font (size 1.27 1.27)) hide)
+    )
+    (property "Value" "GND" (id 1) (at 267.081 190.9572 90)
+      (effects (font (size 1.27 1.27)) (justify right))
+    )
+    (property "Footprint" "" (id 2) (at 266.954 187.706 0)
+      (effects (font (size 1.27 1.27)) hide)
+    )
+    (property "Datasheet" "" (id 3) (at 266.954 187.706 0)
+      (effects (font (size 1.27 1.27)) hide)
+    )
+    (pin "1")
+  )
   (symbol (lib_id "Switch:SW_Push") (at 151.892 145.542 0) (unit 1)
     (in_bom yes) (on_board yes)
@@
       (reference "#PWR0110") (unit 1) (value "GND") (footprint "")
     )
+    (path "/f0efa3ea-26e1-4220-ae1d-41709ae949ef"
+      (reference "#PWR?") (unit 1) (value "GND") (footprint "")
+    )
     (path "/00000000-0000-0000-0000-000060088079"
